File: esp32_dev.kicad_pcb (KiCad board)
At the start: 4 copper layers, 31.2 x 50.1 mm, 35 parts, among them J1 Conn_01x19_Pin, J2 Conn_01x19_Pin, J3 USB_B_Micro, Q1 SS8050, Q2 SS8050, U1 AMS1117-3.3, U3 CP2102N-Axx-xQFN28

Commit message: pcb modified
Other:
- board size 31.2 x 50.1 mm -> 31.2 x 56.8 mm
Changed lines of the file:
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@@
 		(embedded_fonts no)
+	)
+	(gr_line
+		(start 86.375 72.85)
+		(end 86.375 66.4875)
+		(stroke
+			(width 0.05)
+			(type default)
+		)
+		(layer "Edge.Cuts")
 	)
 	(gr_curve
@@
 			(xy 110.3884 122.936) (xy 111.4044 122.936) (xy 111.4044 121.8184) (xy 111.4044 121.7676)
 		)
+		(stroke
+			(width 0.05)
+			(type default)
+		)
+		(layer "Edge.Cuts")
+	)
+	(gr_arc
+		(start 86.375 66.4875)
+		(mid 86.492157 66.204657)
+		(end 86.775 66.0875)
 		(stroke
 			(width 0.05)
@@
 	)
 	(gr_line
+		(start 105.15 66.4875)
+		(end 105.15 72.85)
+		(stroke
+			(width 0.05)
+			(type default)
+		)
+		(layer "Edge.Cuts")
+	)
+	(gr_line
 		(start 80.1624 121.92)
 		(end 80.1624 74.0156)
+		(stroke
+			(width 0.05)
+			(type default)
+		)
+		(layer "Edge.Cuts")
+	)
+	(gr_line
+		(start 105.15 72.85)
+		(end 110.236 72.8472)
+		(stroke
+			(width 0.05)
+			(type default)
+		)
+		(layer "Edge.Cuts")
+	)
+	(gr_line
+		(start 86.775 66.0875)
+		(end 104.75 66.0875)
 		(stroke
 			(width 0.05)
@@
 			(xy 80.1624 121.92) (xy 80.1624 122.936) (xy 81.28 122.936) (xy 81.3308 122.936)
 		)
+		(stroke
+			(width 0.05)
+			(type default)
+		)
+		(layer "Edge.Cuts")
+	)
+	(gr_arc
+		(start 104.75 66.0875)
+		(mid 105.032843 66.204657)
+		(end 105.15 66.4875)
 		(stroke
 			(width 0.05)
@@
 	(gr_line
 		(start 81.1784 72.8472)
-		(end 110.236 72.8472)
+		(end 86.375 72.85)
 		(stroke
 			(width 0.05)
